Commit message: added llm to save waypoint

File: urdf/robot_core.xacro (robot description, xacro)
@@ -7,4 +7,7 @@
     <color rgba="0.00784313725490196 0.8470588235294118 0.9137254901960784 1.0" />
   </material>
+  <material name="black">
+        <color rgba="0.26 0.23 0.25 1.0"/>
+  </material>
   <link name="base_link">
     <inertial>
@@ -19,5 +22,5 @@
         <mesh filename="file:///home/naveen/alpha_bot/src/alpha_bot/meshes/base_link.STL"/>
       </geometry>
-      <material name="red">
+      <material name="orange">
         <color rgba="0.79216 0.81961 0.93333 1"/>
       </material>
@@ -41,6 +44,6 @@
         <mesh filename="file:///home/naveen/alpha_bot/src/alpha_bot/meshes/left_wheel.STL"/>
       </geometry>
-      <material name="">
-        <color rgba="0.64706 0.61961 0.58824 1"/>
+      <material name="black">
+        <color rgba="0.26 0.23 0.25 1.0"/>
       </material>
     </visual>
@@ -70,6 +73,6 @@
         <mesh filename="file:///home/naveen/alpha_bot/src/alpha_bot/meshes/right_wheel.STL"/>
       </geometry>
-      <material name="">
-        <color rgba="0.64706 0.61961 0.58824 1"/>
+      <material name="black">
+        <color rgba="0.26 0.23 0.25 1.0"/>
       </material>
     </visual>
